File: 15x15 Matrix/5x5 Matrix/5x5 Matrix.kicad_sch (KiCad schematic)
At the start: 111 parts, among them J1 Conn_01x02, SW1 SWP, SW10 SWP, SW11 SWP, SW12 SWP, SW13 SWP, SW14 SWP, SW15 SWP, SW16 SWP, SW17 SWP, SW18 SWP, SW19 SWP, SW2 SWP, SW20 SWP, SW21 SWP, SW22 SWP, SW23 SWP, SW24 SWP, SW25 SWP, SW3 SWP, SW4 SWP, SW5 SWP, SW6 SWP, SW7 SWP, SW8 SWP, SW9 SWP, U1 MCP23017x-x-SO, U2 74AHCT1G125

Commit message: Fixed naming for JLC components
Parts:
- D1, D10, D11, D12, D13, D14, D15, D16, D17, D18, D19, D2, D20, D21, D22, D23, D24, D25, D3, D4, D5, D6, D7, D8, D9: value D -> 1N4148W
- U1: value MCP23017x-x-SO -> MCP23017-E/SO
Connections:
- net 5V: now also C27.2, U2.5 (VCC); no longer C27.1
- net GND: now also C27.1
Other:
- moved on the sheet: C26, C27, D10, D12, D13, D14, D15, D17, D18, D19, D2, D20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

Commit message: 5x5 Ready for 1 sided printing
Parts:
- removed CPI1: 100nF, footprints:C14663_C0603, symbol Device:C
- A1, SW1, SW10, SW11, SW12, SW13, SW14, SW15, SW16, SW17, SW18, SW19, SW2, SW20, SW21, SW22, SW23, SW24, SW25, SW3, SW4, SW5, SW6, SW7, SW8, SW9: now left out of the parts list
- C1, C10, C11, C12, C13, C14, C15, C16, C17, C18, C19, C2, C20, C21, C22, C23, C24, C25, C27, C3, C4, C5, C6, C7, C8, C9: LCSC Part # (none) -> C14663
- C26: footprint footprints:C49304896_CAP-TH_BD6_3-P2_50-D0_5-FD -> Capacitor_THT:CP_Radial_D6.3mm_P2.50mm; LCSC Part # (none) -> C49304896
- C28: renamed from CPI2; LCSC Part # (none) -> C14663
- D1, D10, D11, D12, D13, D14, D15, D16, D17, D18, D19, D2, D20, D21, D22, D23, D24, D25, D3, D4, D5, D6, D7, D8, D9: LCSC Part # (none) -> C2828417
- D26, D27, D28, D29, D30, D31, D32, D33, D34, D35, D36, D37, D38, D39, D40, D41, D42, D43, D44, D45, D46, D47, D48, D49, D50: footprint footprints:C5149201_LED-SMD_4P-L3_2-W2_8-LS5_9_SK6812MINI-E -> LED_SMD:LED_SK6812MINI-E_3.2x2.8mm_P1.5mm_ReverseMount; LCSC Part # (none) -> C5149201
- J1: LCSC Part # (none) -> C474906
- R1, R2: LCSC Part # (none) -> C23162
- R3: LCSC Part # (none) -> C105881
- U1: LCSC Part # (none) -> C47023
- U2: LCSC Part # (none) -> C7484
